Commit message: Worked on implementing IKPY to enchance our inverse kinematics caclulations

File: src/kinematics/models/SimpleArmModelforURDF.URDF (robot description, URDF)
Before this commit: robot SimpleArmModelforURDF, 6 links, 5 joints
Joints:
- joint Rev2: type continuous -> revolute
- joint Rev3: type continuous -> revolute
- joint Rev4: type continuous -> revolute
- joint Rev5: type continuous -> revolute
- joint Rev6: type continuous -> revolute
