Commit message: Finalized IKPY methods, and IKPY is ready to replace Kinpy ans the ne faster way of calculating inverse and forward kinematics.

File: src/kinematics/models/XArm.urdf (robot description, URDF)
Before this commit: robot xArm, 7 links, 6 joints
Joints:
- joint arm1: type continuous -> revolute
- joint arm2: type continuous -> revolute
- joint arm3: type continuous -> revolute
- joint arm4: type continuous -> revolute
- joint arm5: type continuous -> revolute

Commit message: Added extra link to XArm file in order to make inverse kinematics work (will be removed)

File: src/kinematics/models/XArm.urdf (robot description, URDF)
Before this commit: robot xArm, 7 links, 6 joints
Links:
- added link link6; visual cylinder length=0.004 radius=0.01
Joints:
- added joint arm6: type revolute, parent link5, child link6, origin xyz=0.0 0.0 0.055 rpy=0.0 0.0 0.0, axis 0 0 1
- joint arm1: type continuous -> revolute
- joint arm2: type continuous -> revolute
- joint arm3: type continuous -> revolute
- joint arm4: type continuous -> revolute
- joint arm5: type continuous -> revolute

Commit message: worked on fixing migrating from kinpy to ikpy for forward/inverse kinematics

File: src/kinematics/models/XArm.urdf (robot description, URDF)
Before this commit: robot xArm, 8 links, 7 joints
Links:
- removed link link6
Joints:
- removed joint arm6
