Commit message: Trying to get arm working, added bounds to urdf and changed serial communication

File: c1c0_object_detection/kinematics/models/SimpleArmModelforURDF.urdf (robot description, URDF)
Before this commit: robot SimpleArmModelforURDF, 6 links, 5 joints
Joints:
- joint Rev2: limit (none) -> lower=0 upper=180
- joint Rev3: limit (none) -> lower=0 upper=3.14
- joint Rev4: limit (none) -> lower=0 upper=6.28
- joint Rev5: limit (none) -> lower=0 upper=3
- joint Rev6: limit (none) -> lower=0 upper=6.28
