Commit message: Blue arm kind of working

File: c1c0_object_detection/kinematics/models/XArm.urdf (robot description, URDF)
Before this commit: robot xArm, 7 links, 6 joints
Joints:
- joint arm1: limit (none) -> lower=-1.57 upper=1.57
- joint arm2: limit (none) -> lower=-1.57 upper=1.57
- joint arm3: limit (none) -> lower=-1.57 upper=1.57
- joint arm4: limit (none) -> lower=-1.57 upper=1.57
- joint arm5: limit (none) -> lower=-1.57 upper=1.57
